Commit message: grasp stage1 initially build

File: env/assets/urdf/frankaLinkerHand_description/robots/frankaLinker.urdf (robot description, URDF)
Before this commit: robot panda, 20 links, 19 joints
Joints:
- joint panda_hand_joint: origin xyz=0 0 0.107 rpy=0 0 -0.785398163397 -> xyz=0 0 0.107 rpy=0 0 3.1415926
